Commit message: Navigation stack base integration

File: StarBabyROS/src/starbaby_description/urdf/starbaby.xacro (robot description, xacro)
@@ -5,4 +5,6 @@
     <xacro:property name="body_height" value="0.280" />
     <xacro:property name="body_ground_spacing" value="0.01" />
+    <xacro:property name="body_corner_side_length" value="0.18"/>
+    <xacro:property name="body_corner_front_length" value="0.09"/>
     <xacro:property name="wheel_length" value="0.037" />
     <xacro:property name="wheel_radius" value="0.0375" />
@@ -19,4 +21,9 @@
     <xacro:property name="lidar_x" value="-0.05" />
     <xacro:property name="lidar_y" value="0.057" />
+    <xacro:property name="sonar_length" value="0.02"/>
+    <xacro:property name="sonar_width" value="0.044"/>
+    <xacro:property name="sonar_height" value="0.02"/>
+    <xacro:property name="sonar_center_height" value="0.028"/>
+    <xacro:property name="sonar_side_height" value="0.036"/>
     <!-- Import all Gazebo-customization elements, including Gazebo colors -->
   	<xacro:include filename="$(find starbaby_description)/urdf/starbaby.gazebo" />
@@ -141,3 +148,53 @@
         <origin xyz="${lidar_x} ${lidar_y} ${body_height / 2 + lidar_height / 2}" rpy="0 0 0"/>
     </joint>
+    <link name="sonar_center_link">
+    	<visual>
+            <!-- <geometry>
+                <box size="${sonar_length} ${sonar_width} ${sonar_height}"/>
+            </geometry>-->
+            <geometry>
+				<mesh filename="package://starbaby_description/meshes/HC-SR04.stl" scale="0.001 0.001 0.001"/>
+			</geometry>
+            <material name="white"/>
+        </visual>
+    </link>
+    <joint name="sonar_center_to_body" type="fixed">
+        <parent link="body_link"/>
+        <child link="sonar_center_link"/>
+        <origin xyz="${body_length / 2 - sonar_length / 2} 0 ${-body_height / 2 + sonar_center_height}" rpy="0 0 0"/>
+    </joint>
+    <link name="sonar_left_link">
+    	<visual>
+            <!-- <geometry>
+                <box size="${sonar_length} ${sonar_width} ${sonar_height}"/>
+            </geometry>-->
+            <geometry>
+				<mesh filename="package://starbaby_description/meshes/HC-SR04.stl" scale="0.001 0.001 0.001"/>
+			</geometry>
+            <material name="white"/>
+        </visual>
+    </link>
+    <joint name="sonar_left_to_body" type="fixed">
+        <parent link="body_link"/>
+        <child link="sonar_left_link"/>
+        <origin xyz="${body_length / 2 - sonar_length} ${body_corner_front_length/2 + sonar_width/2} ${-body_height / 2 + sonar_side_height}"
+        	rpy="0 0 ${atan2(body_length - body_corner_side_length, (body_width-body_corner_front_length)/2)}"/>
+    </joint>
+    <link name="sonar_right_link">
+    	<visual>
+            <!-- <geometry>
+                <box size="${sonar_length} ${sonar_width} ${sonar_height}"/>
+            </geometry>-->
+            <geometry>
+				<mesh filename="package://starbaby_description/meshes/HC-SR04.stl" scale="0.001 0.001 0.001"/>
+			</geometry>
+            <material name="white"/>
+        </visual>
+    </link>
+    <joint name="sonar_right_to_body" type="fixed">
+        <parent link="body_link"/>
+        <child link="sonar_right_link"/>
+        <origin xyz="${body_length / 2 - sonar_length} ${-body_corner_front_length/2 - sonar_width/2} ${-body_height / 2 + sonar_side_height}"
+        	rpy="0 0 ${-atan2(body_length - body_corner_side_length, (body_width-body_corner_front_length)/2)}"/>
+    </joint>
 </robot>
