Commit message: Simulation with kalmann filtered odom & beacons detection

File: StarBabyROS/src/starbaby_gazebo/urdf/RobotCities-2018.xacro (robot description, xacro)
@@ -1,4 +1,8 @@
 <?xml version="1.0"?>
 <robot name="robot_cities_2018" xmlns:xacro="http://ros.org/wiki/xacro">
+	<xacro:property name="world_laser_retro" value="10.0"/>
+    <xacro:property name="beacon_width" value="0.1" />
+    <xacro:property name="beacon_height" value="0.5" />
+	<xacro:property name="beacon_laser_retro" value="100.0"/>
     <link name="world"/>
 	<link name="robot_cities_2018">
@@ -7,5 +11,5 @@
 				<mesh filename="package://starbaby_gazebo/meshes/RobotCities-2018-full.stl" scale="0.001 0.001 0.001"/>
 			</geometry>
-    		<origin xyz="-0.489 -1.522 0.0" rpy="${pi/ 2} 0 ${pi/ 2}"/>
+    		<origin xyz="-1.022 -1.522 0.0" rpy="${pi/ 2} 0 ${pi/ 2}"/>
 		</visual>
 		<collision>
@@ -13,5 +17,6 @@
 				<mesh filename="package://starbaby_gazebo/meshes/RobotCities-2018-full.stl" scale="0.001 0.001 0.001"/>
 			</geometry>
-    		<origin xyz="-0.489 -1.522 0.0" rpy="${pi/ 2} 0 ${pi/ 2}"/>
+    		<origin xyz="-1.022 -1.522 0.0" rpy="${pi/ 2} 0 ${pi/ 2}"/>
+    		<laser_retro>${world_laser_retro}</laser_retro>
 		</collision>
         <inertial>
@@ -25,4 +30,10 @@
 		<material>Gazebo/Orange</material>
 		<static>true</static>
+		<visual>
+    		<laser_retro>${world_laser_retro}</laser_retro>
+		</visual>
+		<collision>
+    		<laser_retro>${world_laser_retro}</laser_retro>
+		</collision>
 	</gazebo>
     <joint name="world_to_robot_cities_2018" type="fixed">
@@ -31,3 +42,41 @@
     	<origin xyz="0 0 0" rpy="0 0 0"/>
 	</joint>
+	<xacro:macro name="beacon" params="beacon_name beacon_x beacon_y">
+		<link name="${beacon_name}">
+			<visual>
+	            <geometry>
+	                <box size="${beacon_width} ${beacon_width} ${beacon_height}"/>
+	            </geometry>
+	    		<origin xyz="0 0 ${beacon_height/2}" rpy="0 0 0"/>
+	            <material name="white"/>
+			</visual>
+			<collision>
+	            <geometry>
+	                <box size="${beacon_width} ${beacon_width} ${beacon_height}"/>
+	            </geometry>
+	    		<origin xyz="0 0 ${beacon_height/2}" rpy="0 0 0"/>
+			</collision>
+	        <inertial>
+				<mass value="0.3"/>
+				<inertia ixx="2e-4" ixy="0.0" ixz="0.0" iyy="2e-4" iyz="0.0" izz="2.5e-4"/>
+	        </inertial>
+        </link>
+        <joint name="robot_cities_2018_to_${beacon_name}" type="fixed">
+		    <parent link="world"/>
+		    <child link="${beacon_name}"/>
+	    	<origin xyz="${beacon_x} ${beacon_y} 0.022" rpy="0 0 0"/>
+		</joint>
+		<gazebo reference="${beacon_name}">
+			<material>Gazebo/White</material>
+			<visual>
+	    		<laser_retro>${beacon_laser_retro}</laser_retro>
+			</visual>
+			<collision>
+	    		<laser_retro>${beacon_laser_retro}</laser_retro>
+			</collision>
+		</gazebo>
+	</xacro:macro>
+	<beacon beacon_name="beacon_1" beacon_x="-0.95" beacon_y="1.594"/>
+	<beacon beacon_name="beacon_2" beacon_x="0.0" beacon_y="-1.594"/>
+	<beacon beacon_name="beacon_3" beacon_x="0.95" beacon_y="1.594"/>
 </robot>

Commit message: Trilateration handles both side of the field & split launch

File: StarBabyROS/src/starbaby_gazebo/urdf/RobotCities-2018.xacro (robot description, xacro)
@@ -5,4 +5,5 @@
     <xacro:property name="beacon_height" value="0.5" />
 	<xacro:property name="beacon_laser_retro" value="100.0"/>
+	<xacro:property name="beacon_side" value="1"/>
     <link name="world"/>
 	<link name="robot_cities_2018">
@@ -77,6 +78,6 @@
 		</gazebo>
 	</xacro:macro>
-	<beacon beacon_name="beacon_1" beacon_x="-0.95" beacon_y="1.594"/>
-	<beacon beacon_name="beacon_2" beacon_x="0.0" beacon_y="-1.594"/>
-	<beacon beacon_name="beacon_3" beacon_x="0.95" beacon_y="1.594"/>
+	<beacon beacon_name="beacon_1" beacon_x="-0.95" beacon_y="${beacon_side * -1.594}"/>
+	<beacon beacon_name="beacon_2" beacon_x="0.0" beacon_y="${beacon_side * 1.594}"/>
+	<beacon beacon_name="beacon_3" beacon_x="0.95" beacon_y="${beacon_side * -1.594}"/>
 </robot>
